Commit message: added gazebo simulation and made a visual of rviz

File: src/staubli/staubli_rx160_support/urdf/gazebo.urdf (robot description, URDF)
Before this commit: robot staubli_rx160, 9 links, 8 joints
Links:
- added link base
- added link flange
Joints:
- removed joint fixed
- removed joint joint_6-tool0
- added joint base_link-base: type fixed, parent base_link, child base, origin xyz=0 0 0.550 rpy=0 0 0
- added joint flange-tool0: type fixed, parent flange, child tool0, origin xyz=0 0 0 rpy=0 1.57079632679 0
- added joint joint_6-flange: type fixed, parent link_6, child flange, origin xyz=0 0 0 rpy=0 -1.57079632679 0
- joint joint_1: limit lower=-2.967060 upper=2.967060 effort=692.0 velocity=2.88 -> lower=-2.79252680319 upper=2.79252680319 effort=692.0 velocity=3.49065850399
- joint joint_2: limit lower=-2.4 upper=2.4 effort=574.0 velocity=2.62 -> lower=-2.39982772149 upper=2.39982772149 effort=574.0 velocity=3.49065850399
- joint joint_3: limit lower=-2.62 upper=2.62 effort=242.0 velocity=3.32 -> lower=-2.61799387799 upper=2.61799387799 effort=242.0 velocity=4.45058959259
- joint joint_4: limit lower=-4.71 upper=4.71 effort=58.0 velocity=5.15 -> lower=-4.71238898038 upper=4.71238898038 effort=58.0 velocity=5.49778714378
- joint joint_5: limit lower=-1.83 upper=2.09 effort=29.0 velocity=4.54 -> lower=-1.83259571459 upper=2.09439510239 effort=29.0 velocity=6.28318530718
- joint joint_6: limit lower=-4.71 upper=4.71 effort=29.0 velocity=7.68 -> lower=-4.71238898038 upper=4.71238898038 effort=29.0 velocity=15.1843644924
